File: processing/processing.kicad_pcb (KiCad board)
At the start: 2 copper layers, 100 x 100 mm, 195 parts, among them J1 Conn_01x08_Male, J2 Conn_01x06_Male, J3 power_amp, J4 control board, J5 AudioJack2_X4, J6 AudioJack2_XLR_SW, J7 Conn_01x03_Male, Q1 TD9944, Q3 MMUN2111LT1, Q4 MMBT2222A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

Commit message: Add processing PCB
Parts:
- removed C37: 2.2µF/25V/UL ESR, Capacitor_SMD:C_0805_2012Metric
- removed R48, R49: 10k, Resistor_SMD:R_0805_2012Metric
- added C56: 2.2µF/25V/UL ESR, Capacitor_SMD:C_0805_2012Metric, F.Cu at (39.1, 66.0)
- added C57: 2.2µF/25V/UL ESR, Capacitor_SMD:C_0805_2012Metric, F.Cu at (50.9, 61.0)
- added C58: 2.2µF/25V/UL ESR, Capacitor_SMD:C_0805_2012Metric, F.Cu at (113.1, 101.0)
- added J8: Conn_01x02_Male, Connector_PinSocket_2.54mm:PinSocket_1x02_P2.54mm_Vertical, F.Cu at (115.0, 108.0)
- added R73: 10k, Resistor_SMD:R_0805_2012Metric, F.Cu at (93.0, 75.0)
- added R74: 10k, Resistor_SMD:R_0805_2012Metric, F.Cu at (93.1, 78.0)
- added RV2: R_POT, Connector_PinSocket_2.54mm:PinSocket_1x03_P2.54mm_Vertical, F.Cu at (66.0, 106.0)
- added U10: TL072, Package_SO:SOIC-8_3.9x4.9mm_P1.27mm, F.Cu at (45.0, 64.0)
- C47, C48, C53, C54: footprint Capacitor_SMD:C_0805_2012Metric -> Capacitor_SMD:C_0603_1608Metric
- C50: value 47µF/10V -> 10µF/10V
- J1: value Conn_01x08_Male -> Conn_01x06_Male; footprint Connector_PinSocket_2.54mm:PinSocket_1x08_P2.54mm_Vertical -> Connector_PinSocket_2.54mm:PinSocket_1x06_P2.54mm_Vertical
- R39: value 10k -> 0
- R40, R41: value 1k -> 10k
- RV1: value 10k -> R_POT; footprint Connector_PinSocket_2.54mm:PinSocket_1x06_P2.54mm_Vertical -> Connector_PinSocket_2.54mm:PinSocket_1x03_P2.54mm_Vertical
- moved R39 152.1 mm to (64.0, 35.9), turned to 90 degrees
- moved R67 129.1 mm to (40.5, 72.1), turned to 90 degrees
- moved TP27 124.6 mm to (100.0, 71.0)
- moved R10 121.8 mm to (32.9, 74.0)
- moved R72 121.3 mm to (29.4, 47.0)
- moved TP31 120.5 mm to (38.0, 58.0)
- moved R52 118.7 mm to (104.0, 72.1), turned to 90 degrees
- moved R50 118.4 mm to (110.0, 72.1), turned to 90 degrees
- moved TP2 115.8 mm to (22.0, 85.0)
- moved R63 114.4 mm to (46.9, 69.0)
- moved R64 114.1 mm to (50.9, 65.0), turned to 180 degrees
- moved TP19 114.0 mm to (80.0, 78.0)
- moved C46 113.7 mm to (37.0, 71.4), turned to 90 degrees
- moved TP11 113.6 mm to (70.0, 76.0)
- moved C38 113.5 mm to (98.0, 77.1), turned to 270 degrees
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Connections:
- J1 pad 5: A+3.3V -> GNDA
- J5 pad 4: Net-(C20-Pad1) -> Net-(C25-Pad1)
- J5 pad 6: Net-(C25-Pad1) -> Net-(C26-Pad1)
- J5 pad 8: Net-(C26-Pad1) -> Net-(C20-Pad1)
- J6 pad 3: Net-(C31-Pad2) -> Net-(C29-Pad1)
- J6 pad 4: Net-(C29-Pad1) -> Net-(C31-Pad2)
- J6 pad 5: Net-(C28-Pad1) -> Net-(C31-Pad2)
- J6 pad 6: Net-(C31-Pad2) -> Net-(C28-Pad1)
- R39 pad 1: Net-(C33-Pad1) -> GNDA
- R39 pad 2: GNDA -> GNDD
- R40 pad 1: /analog/octaver_down/REF+1.65V -> Net-(R40-Pad1)
- R41 pad 2: /analog/octaver_down/REF+1.65V -> Net-(R40-Pad1)
- R42 pad 2: /codec/ADC_input_A -> /analog/octaver_down/half_signal_in
- R45 pad 2: /codec/ADC_input_A -> /analog/octaver_down/half_signal_in
- U2 pad 10: GNDA -> Net-(R21-Pad1)
- U2 pad 12: Net-(RV1-Pad2) -> Net-(RV2-Pad2)
- U2 pad 13: Net-(D6-Pad1) -> Net-(R34-Pad1)
- U2 pad 14: Net-(D6-Pad1) -> /analog/power_amp_signal
- U2 pad 8: Net-(D7-Pad1) -> Net-(R28-Pad1)
- U2 pad 9: Net-(R30-Pad2) -> Net-(R26-Pad1)
- U3 pad 1: Net-(R28-Pad1) -> Net-(D6-Pad1)
- U3 pad 2: Net-(R26-Pad1) -> Net-(D6-Pad1)
- U3 pad 3: Net-(R21-Pad1) -> Net-(RV1-Pad2)
- U3 pad 5: Net-(RV1-Pad5) -> GNDA
- U3 pad 6: Net-(R34-Pad1) -> Net-(R30-Pad2)
- U3 pad 7: /analog/power_amp_signal -> Net-(D7-Pad1)
- U4 pad 10: (no net) -> /analog/octaver_down/REF+1.65V
- U4 pad 12: /analog/octaver_down/REF+1.65V -> Net-(R73-Pad1)
- U4 pad 13: Net-(R42-Pad1) -> /analog/octaver_down/half_signal_in
- U4 pad 14: Net-(R43-Pad1) -> /analog/octaver_down/half_signal_in
- U4 pad 5: Net-(C43-Pad2) -> Net-(R40-Pad1)
- U4 pad 6: Net-(R62-Pad1) -> /analog/octaver_down/REF+1.65V
- U4 pad 7: Net-(C46-Pad2) -> /analog/octaver_down/REF+1.65V
- U4 pad 8: (no net) -> Net-(R43-Pad1)
- U4 pad 9: (no net) -> Net-(R42-Pad1)
- U5 pad 10: /analog/octaver_down/REF+1.65V -> A+3.3V
- U5 pad 12: /analog/octaver_down/REF+1.65V -> A+3.3V
- U6 pad 15: (no net) -> Net-(U6-Pad15)
- U7 pad 3: /codec/ADC_input_A -> /analog/octaver_down/half_signal_in
Routing:
- net A+15V: track 0.00 -> 275.1 mm, vias 0 -> 8
- net A-15V: track 0.00 -> 273.7 mm, vias 0 -> 9
- net A+3.3V: track 0.00 -> 250.5 mm, vias 0 -> 8
- net /SDA: track 0.00 -> 62.6 mm
- net Net-(R21-Pad1): track 0.00 -> 55.3 mm
- net /SCL: track 0.00 -> 54.6 mm, vias 0 -> 1
- net /codec/INB: track 0.00 -> 54.1 mm
- net /analog/octaver_down/half_signal_in: track 0.00 -> 53.5 mm
- net /codec/~MUTEB: track 0.00 -> 52.9 mm
- net Net-(R1-Pad2): track 0.00 -> 49.6 mm, vias 0 -> 2
- net /codec/ADC_input_A: track 0.00 -> 45.4 mm
- net /analog/octaver_down/REF+1.65V: track 0.00 -> 42.6 mm, vias 0 -> 2
- net /codec/OUTB: track 0.00 -> 42.5 mm
- net /codec/INA: track 0.00 -> 41.6 mm
- net /codec/~MUTEA: track 0.00 -> 41.0 mm, vias 0 -> 2
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- added copper zone on B.Cu, net GNDA
- added copper zone on F.Cu, net GNDA
- added copper zone on B.Cu, net GNDD
- added copper zone on F.Cu, net GNDD
