File: electronics/processing/processing.kicad_pcb (KiCad board)
At the start: 2 copper layers, 100 x 100 mm, 200 parts, among them J1 Conn_01x06_Male, J2 Conn_01x06_Male, J3 power_amp, J4 control board, J5 AudioJack2_X4, J6 AudioJack2_XLR_SW, J7 Conn_01x03_Male, J8 Conn_01x02_Male, Q1 TD9944, Q3 MMUN2111LT1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

Commit message: Création des gerber de processing et correction des gerber de psu.
Parts:
- moved C7 64.9 mm to (111.0, 43.1), turned to 90 degrees
- moved J8 64.0 mm to (116.0, 44.0)
- moved C3 63.4 mm to (113.0, 51.0), turned to 270 degrees
Routing:
- net A+3.3V: track 250.5 -> 260.4 mm
- net GNDA: vias 113 -> 112
Other:
- board text added: "(G/S) In/Tuner/Send/Return"
- board text added: "2xA+15/2xA-15/2xG"
- board text added: "3xD+5/3xG"
- board text added: "A+3.3/G"
- board text added: "Direct out vol"
- board text added: "G lift/XLR/Jack"
- board text added: "Gain/Pad"
- board text added: "Power Vol"
- board text added: "Power amp"
- board text added: "S/~Mute~/G"
- board text added: "TX/RX/G"
Changed lines of the file:
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@@
-(kicad_pcb (version 20171130) (host pcbnew 5.1.5-52549c5~84~ubuntu18.04.1)
+(kicad_pcb (version 20171130) (host pcbnew 5.1.5+dfsg1-2build2)
   (general
     (thickness 1.6)
-    (drawings 6)
+    (drawings 17)
     (tracks 1127)
     (zones 0)
@@
   )
   (setup
-    (last_trace_width 0.25)
+    (last_trace_width 1.27)
     (user_trace_width 0.254)
     (user_trace_width 0.508)
@@
     (visible_elements FFFDFF7F)
     (pcbplotparams
-      (layerselection 0x010fc_ffffffff)
-      (usegerberextensions false)
+      (layerselection 0x010f0_ffffffff)
+      (usegerberextensions true)
       (usegerberattributes false)
       (usegerberadvancedattributes false)
@@
       (outputformat 1)
       (mirror false)
-      (drillshape 1)
+      (drillshape 0)
       (scaleselection 1)
       (outputdirectory ""))
@@
   )
   (module Connector_PinSocket_2.54mm:PinSocket_1x02_P2.54mm_Vertical (layer F.Cu)
-    (at 115 108 180)
+    (at 116 44 180)
     (descr "Through hole straight socket strip, 1x02, 2.54mm pitch, single row (from Kicad 4.0.7), script generated")
     (tags "Through hole socket strip THT 1x02 2.54mm single row")
@@
   )
   (module Capacitor_SMD:C_0805_2012Metric (layer F.Cu)
-    (at 111.0625 108 180)
+    (at 111 43.0625 90)
     (descr "Capacitor SMD 0805 (2012 Metric), square (rectangular) end terminal, IPC_7351 nominal, (Body size source: https://docs.google.com/spreadsheets/d/1BsfQQcO9C6DZCsRaXUlFlo91Tg2WpOkGARC1WS5S8t0/edit?usp=sharing), generated with kicad-footprint-generator")
     (tags capacitor)
     (attr smd)
-    (fp_text reference C7 (at 0 2) (layer F.SilkS)
+    (fp_text reference C7 (at 0.0625 -2 90) (layer F.SilkS)
       (effects (font (size 1 1) (thickness 0.15)))
     )
-    (fp_text value "2.2µF/25V/UL ESR" (at 0 1.65) (layer F.Fab)
+    (fp_text value "2.2µF/25V/UL ESR" (at 0 1.65 90) (layer F.Fab)
       (effects (font (size 1 1) (thickness 0.15)))
     )
-    (fp_text user %R (at 0 0) (layer F.Fab)
+    (fp_text user %R (at 0 0 90) (layer F.Fab)
       (effects (font (size 0.5 0.5) (thickness 0.08)))
     )
@@
     (fp_line (start -1 -0.6) (end 1 -0.6) (layer F.Fab) (width 0.1))
     (fp_line (start -1 0.6) (end -1 -0.6) (layer F.Fab) (width 0.1))
-    (pad 2 smd roundrect (at 0.9375 0 180) (size 0.975 1.4) (layers F.Cu F.Paste F.Mask) (roundrect_rratio 0.25)
+    (pad 2 smd roundrect (at 0.9375 0 90) (size 0.975 1.4) (layers F.Cu F.Paste F.Mask) (roundrect_rratio 0.25)
       (net 1 GNDA))
-    (pad 1 smd roundrect (at -0.9375 0 180) (size 0.975 1.4) (layers F.Cu F.Paste F.Mask) (roundrect_rratio 0.25)
+    (pad 1 smd roundrect (at -0.9375 0 90) (size 0.975 1.4) (layers F.Cu F.Paste F.Mask) (roundrect_rratio 0.25)
       (net 4 A+3.3V))
     (model ${KISYS3DMOD}/Capacitor_SMD.3dshapes/C_0805_2012Metric.wrl
@@
   )
   (module Capacitor_THT:CP_Radial_D10.0mm_P5.00mm (layer F.Cu)
-    (at 106 114 180)
+    (at 113 51 270)
     (descr "CP, Radial series, Radial, pin pitch=5.00mm, , diameter=10mm, Electrolytic Capacitor")
     (tags "CP Radial series Radial pin pitch 5.00mm  diameter 10mm Electrolytic Capacitor")
-    (fp_text reference C3 (at 2.5 6) (layer F.SilkS)
+    (fp_text reference C3 (at 2.5 6 90) (layer F.SilkS)
       (effects (font (size 1 1) (thickness 0.15)))
     )
-    (fp_text value 1000µF/25V (at 2.5 6.25) (layer F.Fab)
+    (fp_text value 1000µF/25V (at 2.5 6.25 90) (layer F.Fab)
       (effects (font (size 1 1) (thickness 0.15)))
     )
-    (fp_text user %R (at 2.5 0) (layer F.Fab)
+    (fp_text user %R (at 2.5 0 90) (layer F.Fab)
       (effects (font (size 1 1) (thickness 0.15)))
     )
@@
     (fp_circle (center 2.5 0) (end 7.62 0) (layer F.SilkS) (width 0.12))
     (fp_circle (center 2.5 0) (end 7.5 0) (layer F.Fab) (width 0.1))
-    (pad 2 thru_hole circle (at 5 0 180) (size 2 2) (drill 1) (layers *.Cu *.Mask)
+    (pad 2 thru_hole circle (at 5 0 270) (size 2 2) (drill 1) (layers *.Cu *.Mask)
       (net 1 GNDA))
-    (pad 1 thru_hole rect (at 0 0 180) (size 2 2) (drill 1) (layers *.Cu *.Mask)
+    (pad 1 thru_hole rect (at 0 0 270) (size 2 2) (drill 1) (layers *.Cu *.Mask)
       (net 4 A+3.3V))
     (model ${KISYS3DMOD}/Capacitor_THT.3dshapes/CP_Radial_D10.0mm_P5.00mm.wrl
@@
     )
   )
+  (gr_text S/~Mute~/G (at 80 21) (layer F.SilkS)
+    (effects (font (size 1 1) (thickness 0.15)))
+  )
+  (gr_text TX/RX/G (at 64 21) (layer F.SilkS)
+    (effects (font (size 1 1) (thickness 0.15)))
+  )
+  (gr_text 3xD+5/3xG (at 49 21) (layer F.SilkS)
+    (effects (font (size 1 1) (thickness 0.15)))
+  )
+  (gr_text A+3.3/G (at 119 43 90) (layer F.SilkS)
+    (effects (font (size 1 1) (thickness 0.15)))
+  )
+  (gr_text "G lift/XLR/Jack" (at 83 119) (layer F.SilkS)
+    (effects (font (size 1 1) (thickness 0.15)))
+  )
+  (gr_text Gain/Pad (at 63 78 270) (layer F.SilkS)
+    (effects (font (size 1 1) (thickness 0.15)))
+  )
+  (gr_text "Direct out vol" (at 77 90) (layer F.SilkS)
+    (effects (font (size 1 1) (thickness 0.15)))
+  )
+  (gr_text "Power Vol" (at 69 103 270) (layer F.SilkS)
+    (effects (font (size 1 1) (thickness 0.15)))
+  )
+  (gr_text "Power amp" (at 69 93 270) (layer F.SilkS)
+    (effects (font (size 1 1) (thickness 0.15)))
+  )
+  (gr_text 2xA+15/2xA-15/2xG (at 62 119) (layer F.SilkS)
+    (effects (font (size 1 1) (thickness 0.15)))
+  )
+  (gr_text "(G/S) In/Tuner/Send/Return" (at 30 92 270) (layer F.SilkS)
+    (effects (font (size 1 1) (thickness 0.15)))
+  )
   (gr_line (start 120 70) (end 115 70) (layer F.SilkS) (width 0.15))
   (gr_line (start 20 70) (end 25 70) (layer F.SilkS) (width 0.15))
@@
   (via (at 117 92) (size 0.8) (drill 0.4) (layers F.Cu B.Cu) (net 1))
   (via (at 114 101) (size 0.8) (drill 0.4) (layers F.Cu B.Cu) (net 1))
-  (via (at 110 108) (size 0.8) (drill 0.4) (layers F.Cu B.Cu) (net 1))
   (via (at 107 71) (size 0.8) (drill 0.4) (layers F.Cu B.Cu) (net 1))
   (via (at 107 85) (size 0.8) (drill 0.4) (layers F.Cu B.Cu) (net 1))
@@
   (segment (start 78 101) (end 78 101) (width 0.508) (layer F.Cu) (net 3))
   (via (at 78 101) (size 0.8) (drill 0.4) (layers F.Cu B.Cu) (net 3))
-  (segment (start 78 101) (end 75 104) (width 0.508) (layer B.Cu) (net 3))
+  (segment (start 75 104) (end 78 101) (width 1.27) (layer B.Cu) (net 3))
   (segment (start 80.125 87) (end 78 87) (width 0.508) (layer F.Cu) (net 4))
   (segment (start 77 81.125) (end 74 81.125) (width 0.508) (layer F.Cu) (net 4))
@@
   (segment (start 111.49 100.365) (end 112.125 101) (width 0.508) (layer F.Cu) (net 4))
   (segment (start 109.475 100.365) (end 111.49 100.365) (width 0.508) (layer F.Cu) (net 4))
-  (segment (start 115 108) (end 112 108) (width 1.27) (layer F.Cu) (net 4))
-  (segment (start 112 108.7) (end 112 108) (width 1.27) (layer F.Cu) (net 4))
-  (segment (start 112 110.27) (end 112 108.7) (width 1.27) (layer F.Cu) (net 4))
-  (segment (start 108.27 114) (end 112 110.27) (width 1.27) (layer F.Cu) (net 4))
-  (segment (start 106 114) (end 108.27 114) (width 1.27) (layer F.Cu) (net 4))
   (segment (start 112 101.125) (end 112.125 101) (width 1.27) (layer F.Cu) (net 4))
-  (segment (start 112 108) (end 112 101.125) (width 1.27) (layer F.Cu) (net 4))
   (segment (start 115 92.7) (end 115 92) (width 1.27) (layer F.Cu) (net 4))
   (segment (start 115 94.827802) (end 115 92.7) (width 1.27) (layer F.Cu) (net 4))
@@
   (segment (start 43.65 44.025) (end 44.10401 43.57099) (width 0.508) (layer F.Cu) (net 4))
   (segment (start 43.65 44.5) (end 43.65 44.025) (width 0.508) (layer F.Cu) (net 4))
+  (segment (start 116 44) (end 111 44) (width 1.27) (layer F.Cu) (net 4))
+  (segment (start 116 48) (end 113 51) (width 1.27) (layer F.Cu) (net 4))
+  (segment (start 116 44) (end 116 48) (width 1.27) (layer F.Cu) (net 4))
+  (segment (start 108 62.796646) (end 108 64) (width 1.27) (layer F.Cu) (net 4))
+  (segment (start 108 53.73) (end 108 62.796646) (width 1.27) (layer F.Cu) (net 4))
+  (segment (start 110.73 51) (end 108 53.73) (width 1.27) (layer F.Cu) (net 4))
+  (segment (start 113 51) (end 110.73 51) (width 1.27) (layer F.Cu) (net 4))
   (via (at 64 35) (size 0.8) (drill 0.4) (layers F.Cu B.Cu) (net 5))
   (via (at 43 30) (size 0.8) (drill 0.4) (layers F.Cu B.Cu) (net 5))
